File: schematics/Digimatic USB Adaptor.kicad_sch (KiCad schematic)
At the start: 4 parts, among them J1 70246, Q1 2N3904, U1 RP2040

Commit message: Blink LED on activity
Parts:
- added D1: LED, symbol Device:LED
Connections:
- net GND: now also D1.1 (K)
- net at U1.37 (GPIO25): now also D1.2 (A)
Changed lines of the file:
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@@
+	(wire
+		(pts
+			(xy 100.33 105.41) (xy 100.33 106.68)
+		)
+		(stroke
+			(width 0)
+			(type default)
+		)
+	)
 	(wire
 		(pts
@@
 	(wire
 		(pts
+			(xy 99.06 105.41) (xy 100.33 105.41)
+		)
+		(stroke
+			(width 0)
+			(type default)
+		)
+	)
+	(wire
+		(pts
 			(xy 85.09 54.61) (xy 91.44 54.61)
 		)
@@
 	(wire
 		(pts
+			(xy 85.09 105.41) (xy 91.44 105.41)
+		)
+		(stroke
+			(width 0)
+			(type default)
+		)
+	)
+	(wire
+		(pts
 			(xy 140.97 40.64) (xy 140.97 49.53)
 		)
@@
 		)
 	)
-	(text_box "Don't know the right connector but Molex 70246 series fits."
-		(exclude_from_sim no)
-		(at 138.43 50.8 0)
-		(size 21.59 8.89)
+	(text_box "Pico default LED.\nNot required."
+		(exclude_from_sim no)
+		(at 104.14 101.6 0)
+		(size 19.05 6.35)
 		(stroke
 			(width 0)
@@
 		)
 	)
-	(label "~{REQ}"
-		(at 85.09 54.61 0)
-		(fields_autoplaced yes)
+	(text_box "Don't know the right connector but Molex 70246 series fits."
+		(exclude_from_sim no)
+		(at 138.43 50.8 0)
+		(size 21.59 8.89)
+		(stroke
+			(width 0)
+			(type default)
+		)
+		(fill
+			(type none)
+		)
 		(effects
 			(font
 				(size 1.27 1.27)
 			)
-			(justify left bottom)
-		)
-	)
-	(label "DATA"
-		(at 85.09 49.53 0)
+			(justify left top)
+		)
+	)
+	(label "~{REQ}"
+		(at 85.09 54.61 0)
 		(fields_autoplaced yes)
 		(effects
@@
 		)
 	)
-	(label "~{CK}"
-		(at 85.09 52.07 0)
+	(label "DATA"
+		(at 85.09 49.53 0)
 		(fields_autoplaced yes)
 		(effects
@@
 			)
 			(justify left bottom)
+		)
+	)
+	(label "~{CK}"
+		(at 85.09 52.07 0)
+		(fields_autoplaced yes)
+		(effects
+			(font
+				(size 1.27 1.27)
+			)
+			(justify left bottom)
+		)
+	)
+	(symbol
+		(lib_id "power:GND")
+		(at 100.33 106.68 0)
+		(unit 1)
+		(exclude_from_sim no)
+		(in_bom yes)
+		(on_board yes)
+		(dnp no)
+		(fields_autoplaced yes)
+		(property "Reference" "#PWR01"
+			(at 100.33 113.03 0)
+			(effects
+				(font
+					(size 1.27 1.27)
+				)
+				(hide yes)
+			)
+		)
+		(property "Value" "GND"
+			(at 100.33 111.76 0)
+			(effects
+				(font
+					(size 1.27 1.27)
+				)
+			)
+		)
+		(property "Footprint" ""
+			(at 100.33 106.68 0)
+			(effects
+				(font
+					(size 1.27 1.27)
+				)
+				(hide yes)
+			)
+		)
+		(property "Datasheet" ""
+			(at 100.33 106.68 0)
+			(effects
+				(font
+					(size 1.27 1.27)
+				)
+				(hide yes)
+			)
+		)
+		(property "Description" "Power symbol creates a global label with name \"GND\" , ground"
+			(at 100.33 106.68 0)
+			(effects
+				(font
+					(size 1.27 1.27)
+				)
+				(hide yes)
+			)
+		)
+		(pin "1"
+		)
+		(instances
+			(project "Digimatic USB Adaptor"
+				(path "/83329baf-d83f-48a5-bb2e-14bf6dbfbbb0"
+					(reference "#PWR01")
+					(unit 1)
+				)
+			)
 		)
 	)
@@
 					(unit 1)
 				)
+			)
+		)
+	)
+	(symbol
+		(lib_id "Device:LED")
+		(at 95.25 105.41 180)
+		(unit 1)
+		(exclude_from_sim no)
+		(in_bom yes)
+		(on_board yes)
+		(dnp no)
+		(fields_autoplaced yes)
+		(property "Reference" "D1"
+			(at 96.8375 97.79 0)
+			(effects
+				(font
+					(size 1.27 1.27)
+				)
+			)
+		)
+		(property "Value" "LED"
+			(at 96.8375 100.33 0)
+			(effects
+				(font
+					(size 1.27 1.27)
+				)
+			)
+		)
+		(property "Footprint" ""
+			(at 95.25 105.41 0)
+			(effects
+				(font
+					(size 1.27 1.27)
+				)
+				(hide yes)
+			)
+		)
+		(property "Datasheet" "~"
+			(at 95.25 105.41 0)
+			(effects
+				(font
+					(size 1.27 1.27)
+				)
+				(hide yes)
+			)
+		)
+		(property "Description" "Light emitting diode"
+			(at 95.25 105.41 0)
+			(effects
+				(font
+					(size 1.27 1.27)
+				)
+				(hide yes)
+			)
+		)
+		(pin "2"
+		)
+		(pin "1"
+		)
+		(instances
+			(project "Digimatic USB Adaptor"
+				(path "/83329baf-d83f-48a5-bb2e-14bf6dbfbbb0"
+					(reference "D1")
+					(unit 1)
+				)
